File: ESP32-LoRA-ADIO/ESP32-LoRA-ADIO.kicad_sch (KiCad schematic)
At the start: 30 parts, among them J1 USB_B_Micro, J2 External Power, J3 AIO/I2C, J4 DIO, J5 RXTX+Power, J6 SMA, J7 JTAG Debugging, Q1 IRLML5203, Q2 2N7002, Q3 2N7002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

Commit message: Replaced the Micro USB connector by a vertical one
Parts:
- J1: footprint Connector_USB:USB_Micro-B_Molex-105017-0001 -> USB3140-30-0230-1-C_REVE1:GCT_USB3140-30-0230-1-C_REVE1
Changed lines of the file:
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@@
     (property "Reference" "J1" (id 0) (at 21.59 44.45 0))
     (property "Value" "USB_B_Micro" (id 1) (at 21.59 46.99 0))
-    (property "Footprint" "Connector_USB:USB_Micro-B_Molex-105017-0001" (id 2) (at 25.4 58.42 0)
+    (property "Footprint" "USB3140-30-0230-1-C_REVE1:GCT_USB3140-30-0230-1-C_REVE1" (id 2) (at 25.4 58.42 0)
       (effects (font (size 1.27 1.27)) hide)
     )
@@
     )
     (path "/6a33cda9-f8ec-49d5-99d6-fd9061f65ca9"
-      (reference "J1") (unit 1) (value "USB_B_Micro") (footprint "Connector_USB:USB_Micro-B_Molex-105017-0001")
+      (reference "J1") (unit 1) (value "USB_B_Micro") (footprint "USB3140-30-0230-1-C_REVE1:GCT_USB3140-30-0230-1-C_REVE1")
     )
     (path "/e098da95-a45b-4e22-a9bd-4cfc0a054c71"
